File: EuroCard Backplane.sch (EAGLE design)
At the start: 20 parts, among them X1 FAC64S, X2 FAC64S, X3 FAC64S, X4 FAC64S, X5 FAC64S, X6 FAC64S, X7 FAC64S, X8 FAC64S

Commit message: Add a couple dimensions to board
Parts:
- removed U$1, U$10, U$11, U$12, U$2, U$3, U$4, U$5, U$6, U$7, U$8, U$9: BACKPLANE, Eurocard-Backplane-jqi:BACKPLANE
Changed lines of the file:
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@@
 <part name="X7" library="Eurocard-Backplane-jqi" deviceset="FAC64S" device=""/>
 <part name="X8" library="Eurocard-Backplane-jqi" deviceset="FAC64S" device=""/>
-<part name="U$1" library="Eurocard-Backplane-jqi" deviceset="BACKPLANE" device=""/>
-<part name="U$2" library="Eurocard-Backplane-jqi" deviceset="BACKPLANE" device=""/>
-<part name="U$3" library="Eurocard-Backplane-jqi" deviceset="BACKPLANE" device=""/>
-<part name="U$4" library="Eurocard-Backplane-jqi" deviceset="BACKPLANE" device=""/>
-<part name="U$5" library="Eurocard-Backplane-jqi" deviceset="BACKPLANE" device=""/>
-<part name="U$6" library="Eurocard-Backplane-jqi" deviceset="BACKPLANE" device=""/>
-<part name="U$7" library="Eurocard-Backplane-jqi" deviceset="BACKPLANE" device=""/>
-<part name="U$8" library="Eurocard-Backplane-jqi" deviceset="BACKPLANE" device=""/>
-<part name="U$9" library="Eurocard-Backplane-jqi" deviceset="BACKPLANE" device=""/>
-<part name="U$10" library="Eurocard-Backplane-jqi" deviceset="BACKPLANE" device=""/>
-<part name="U$11" library="Eurocard-Backplane-jqi" deviceset="BACKPLANE" device=""/>
-<part name="U$12" library="Eurocard-Backplane-jqi" deviceset="BACKPLANE" device=""/>
 </parts>
 <sheets>
