File: EurocardBackplane-V1_0.brd (EAGLE design)
At the start: 426.7 x 129.8 mm, 32 parts, among them IC1 LM399H, J1 JUMPER, U1 MIC5209, U2 WIZ820IO, U3 MIC5209-3.3YS, X1 FAC64S, X10 FAC64S, X11 FAC64S, X21 FAC64S, X4 FAC64S, X5 FAC64S, X7 FAC64S, X7_AUX FAC64S, X8 FAC64S, X9 FAC64S

Commit message: Halfway done adding more connectors
Parts:
- removed X1, X10, X11, X21, X8: FAC64S, Eurocard-Backplane-jqi:FAC64S
- added X0, X1_AUX, X2, X3_AUX, X6: FAC64S, Eurocard-Backplane-jqi:FAC64S
- moved X9 523.8 mm to (383.5, 64.9)
- moved X7 377.1 mm to (322.6, 64.9)
- moved X4 207.8 mm to (139.7, 64.9)
- moved X5 121.9 mm to (200.7, 64.9)
- renumbered X7_AUX to X8_AUX
Connections:
- removed net A1: X11.A2
- removed net A10: X11.A16
- removed net A100: X9.A9
- removed net A101: X9.A15
- removed net A102: X9.A16
- removed net A113: X10.A2
- removed net A114: X10.A5
- removed net A115: X10.A8
- removed net A116: X10.A9
- removed net A117: X10.A15
- removed net A118: X10.A16
- removed net A3: X11.A5
- removed net A33: X21.A2
- removed net A34: X21.A5
- removed net A35: X21.A8
- removed net A36: X21.A9
- removed net A37: X21.A15
- removed net A38: X21.A16
- removed net A4: X11.A8
- removed net A49: X4.A2
- removed net A50: X4.A5
- removed net A51: X4.A8
- removed net A52: X4.A9
- removed net A53: X4.A15
- removed net A54: X4.A16
- removed net A6: X11.A9
- removed net A65: X7.A2
- removed net A66: X7.A5
- removed net A67: X7.A8
- removed net A68: X7.A9
- removed net A69: X7.A15
- removed net A7: X11.A15
- removed net A70: X7.A16
- removed net A81: X8.A2
- removed net A82: X8.A5
- removed net A83: X8.A8
- removed net A84: X8.A9
- removed net A85: X8.A15
- removed net A86: X8.A16
- removed net A97: X9.A2
- removed net A98: X9.A5
- removed net A99: X9.A8
- removed net C1: X11.C2
- removed net C10: X11.C16
- removed net C100: X9.C9
- removed net C101: X9.C15
- removed net C102: X9.C16
- removed net C113: X10.C2
- removed net C114: X10.C5
- removed net C115: X10.C8
- removed net C116: X10.C9
- removed net C117: X10.C15
- removed net C118: X10.C16
- removed net C3: X11.C5
- removed net C33: X21.C2
- removed net C34: X21.C5
- removed net C35: X21.C8
- removed net C36: X21.C9
- removed net C37: X21.C15
- removed net C38: X21.C16
- removed net C4: X11.C8
- removed net C49: X4.C2
- removed net C50: X4.C5
- removed net C51: X4.C8
- removed net C52: X4.C9
- removed net C53: X4.C15
- removed net C54: X4.C16
- removed net C6: X11.C9
- removed net C65: X7.C2
- removed net C66: X7.C5
- removed net C67: X7.C8
- removed net C68: X7.C9
- removed net C69: X7.C15
- removed net C7: X11.C15
- removed net C70: X7.C16
- removed net C81: X8.C2
- removed net C82: X8.C5
- removed net C83: X8.C8
- removed net C84: X8.C9
- removed net C85: X8.C15
- removed net C86: X8.C16
- removed net C97: X9.C2
- removed net C98: X9.C5
- removed net C99: X9.C8
- removed net D10: X21.C10
- removed net D11: X21.C11
- removed net D12: X4.A10
- removed net D13: X4.A11
- removed net D14: X4.C10
- removed net D15: X4.C11
- removed net D16: X7.A10
- removed net D17: X7.A11
- removed net D18: X7.C10
- removed net D19: X7.C11
- removed net D20: X8.A10
- removed net D21: X8.A11
- removed net D22: X8.C10
- removed net D23: X8.C11
- removed net D24: X9.A10
- removed net D25: X9.A11
- removed net D26: X9.C10
- removed net D27: X9.C11
- removed net D28: X10.A10
- removed net D29: X10.A11
- removed net D30: X10.C10
- removed net D31: X10.C11
- removed net D4: X11.A10
- removed net D5: X11.A11
- removed net D6: X11.C10
- removed net D7: X11.C11
- removed net D8: X21.A10
- removed net D9: X21.A11
- removed net GPIO10: X11.A6
- removed net GPIO11: X11.A7
- removed net GPIO12: X11.C3
- removed net GPIO13: X11.C4
- removed net GPIO14: X11.C6
- removed net GPIO15: X11.C7
- removed net GPIO16: X21.A3
- removed net GPIO17: X21.A4
- removed net GPIO18: X21.A6
- removed net GPIO19: X21.A7
- removed net GPIO20: X21.C3
- removed net GPIO21: X21.C4
- removed net GPIO22: X21.C6
- removed net GPIO23: X21.C7
- removed net GPIO24: X4.A3
- removed net GPIO25: X4.A4
- removed net GPIO26: X4.A6
- removed net GPIO27: X4.A7
- removed net GPIO28: X4.C3
- removed net GPIO29: X4.C4
- removed net GPIO30: X4.C6
- removed net GPIO31: X4.C7
- removed net GPIO32: X7.A3
- removed net GPIO33: X7.A4
- removed net GPIO34: X7.A6
- removed net GPIO35: X7.A7
- removed net GPIO36: X7.C3
- removed net GPIO37: X7.C4
- removed net GPIO38: X7.C6
- removed net GPIO39: X7.C7
- removed net GPIO40: X8.A3
- removed net GPIO41: X8.A4
- removed net GPIO42: X8.A6
- removed net GPIO43: X8.A7
- removed net GPIO44: X8.C3
- removed net GPIO45: X8.C4
- removed net GPIO46: X8.C6
- removed net GPIO47: X8.C7
- removed net GPIO48: X9.A3
- removed net GPIO49: X9.A4
- removed net GPIO50: X9.A6
- removed net GPIO51: X9.A7
- removed net GPIO52: X9.C3
- removed net GPIO53: X9.C4
- removed net GPIO54: X9.C6
- removed net GPIO55: X9.C7
- removed net GPIO56: X10.A3
- removed net GPIO58: X10.A6
- removed net GPIO59: X10.A7
- removed net GPIO60: X10.C3
- removed net GPIO62: X10.C6
- removed net GPIO63: X10.C7
- removed net GPIO8: X11.A3
- removed net GPIO9: X11.A4
- removed net I2C_SCL1: X11.C14
- removed net I2C_SCL2: X21.C14
- removed net I2C_SCL3: X4.C14
- removed net I2C_SCL4: X7.C14
- removed net I2C_SCL5: X8.C14
- removed net I2C_SCL6: X9.C14
- removed net I2C_SCL7: X10.C14
- removed net I2C_SDA1: X11.A14
- removed net I2C_SDA2: X21.A14
- removed net I2C_SDA3: X4.A14
- removed net I2C_SDA4: X7.A14
- removed net I2C_SDA5: X8.A14
- removed net I2C_SDA6: X9.A14
- removed net I2C_SDA7: X10.A14
- removed net SPI_C0: TEENSY.27
- removed net SPI_CS1: TEENSY.28
- removed net SPI_CS3: TEENSY.30
- removed net SPI_CS7_AUX: TEENSY.25, X8_AUX.C12
- removed net SPI_MISO1: X11.C13
- removed net SPI_MISO2: X21.C13
- removed net SPI_MISO3: X4.C13
- removed net SPI_MISO4: X7.C13
- removed net SPI_MISO5: X8.C13
- removed net SPI_MISO6: X9.C13
- removed net SPI_MISO7: X10.C13
- removed net SPI_MOSI1: X11.A13
- removed net SPI_MOSI2: X21.A13
- removed net SPI_MOSI3: X4.A13
- removed net SPI_MOSI4: X7.A13
- removed net SPI_MOSI5: X8.A13
- removed net SPI_MOSI6: X9.A13
- removed net SPI_MOSI7: X10.A13
- removed net SPI_SCLK1: X11.A12
- removed net SPI_SCLK2: X21.A12
- removed net SPI_SCLK3: X4.A12
- removed net SPI_SCLK4: X7.A12
- removed net SPI_SCLK5: X8.A12
- removed net SPI_SCLK6: X9.A12
- removed net SPI_SCLK7: X10.A12
- new net SPI_CS0: TEENSY.24, X0.C12
- new net SPI_CS1_AUX: TEENSY.25, X1_AUX.C12
- new net SPI_CS3_AUX: TEENSY.27, X3_AUX.C12
- new net SPI_CS7: TEENSY.31, X7.C12
- new net SPI_CS8_AUX: TEENSY.32, X8_AUX.C12
- new net SPI_CS9: TEENSY.33, X9.C12
- net +15V: now also X7.A31, X7.C31, X9.A31, X9.C31; no longer X1.A31, X1.C31, X5.A31, X5.C31
- net +15V1: now also X6.A31, X6.C31; no longer X11.A31, X11.C31
- net +15V2: now also X5.A31, X5.C31; no longer X21.A31, X21.C31
- net +15V4: now also X3_AUX.A31, X3_AUX.C31; no longer X7.A31, X7.C31
- net +15V5: now also X2.A31, X2.C31; no longer X8.A31, X8.C31
- net +15V6: now also X1_AUX.A31, X1_AUX.C31; no longer X9.A31, X9.C31
- net +15V7: now also X0.A31, X0.C31; no longer X10.A31, X10.C31
- net -15V: now also X7.A30, X7.C30, X9.A30, X9.C30; no longer X1.A30, X1.C30, X5.A30, X5.C30
- net -15V1: now also X6.A30, X6.C30; no longer X11.A30, X11.C30
- net -15V2: now also X5.A30, X5.C30; no longer X21.A30, X21.C30
- net -15V4: now also X3_AUX.A30, X3_AUX.C30; no longer X7.A30, X7.C30
- net -15V5: now also X2.A30, X2.C30; no longer X8.A30, X8.C30
- net -15V6: now also X1_AUX.A30, X1_AUX.C30; no longer X9.A30, X9.C30
- net -15V7: now also X0.A30, X0.C30; no longer X10.A30, X10.C30
- net A103: now also X1_AUX.A17; no longer X9.A17
- net A104: now also X1_AUX.A18; no longer X9.A18
- net A105: now also X1_AUX.A19; no longer X9.A19
- net A106: now also X1_AUX.A20; no longer X9.A20
- net A107: now also X1_AUX.A21; no longer X9.A21
- net A108: now also X1_AUX.A22; no longer X9.A22
- net A109: now also X1_AUX.A23; no longer X9.A23
- net A11: now also X6.A17; no longer X11.A17
- net A110: now also X1_AUX.A27; no longer X9.A27
- net A111: now also X1_AUX.A28; no longer X9.A28
- net A112: now also X1_AUX.A29; no longer X9.A29
- net A119: now also X0.A17; no longer X10.A17
- net A12: now also X6.A18; no longer X11.A18
- net A120: now also X0.A18; no longer X10.A18
- net A121: now also X0.A19; no longer X10.A19
- net A122: now also X0.A20; no longer X10.A20
- net A123: now also X0.A21; no longer X10.A21
- net A124: now also X0.A22; no longer X10.A22
- net A125: now also X0.A23; no longer X10.A23
- net A126: now also X0.A27; no longer X10.A27
- net A127: now also X0.A28; no longer X10.A28
- net A128: now also X0.A29; no longer X10.A29
- net A13: now also X6.A19; no longer X11.A19
- net A14: now also X6.A20; no longer X11.A20
- net A15: now also X0.A15, X1_AUX.A15, X2.A15, X3_AUX.A15, X4.A15, X6.A15, X7.A15, X9.A15; no longer X1.A15
- net A16: now also X0.A16, X1_AUX.A16, X2.A16, X3_AUX.A16, X4.A16, X6.A16, X7.A16, X9.A16; no longer X1.A16
- net A17: now also X7.A17, X9.A17; no longer X1.A17, X5.A17
- net A18: now also X7.A18, X9.A18; no longer X1.A18, X5.A18
- net A19: now also X7.A19, X9.A19; no longer X1.A19, X5.A19
- net A2: now also X0.A2, X1_AUX.A2, X2.A2, X3_AUX.A2, X4.A2, X6.A2, X7.A2, X9.A2; no longer X1.A2
- net A20: now also X7.A20, X9.A20; no longer X1.A20, X5.A20
- net A21: now also X7.A21, X9.A21; no longer X1.A21, X5.A21
- net A22: now also X7.A22, X9.A22; no longer X1.A22, X5.A22
- net A23: now also X7.A23, X9.A23; no longer X1.A23, X5.A23
- net A24: now also X6.A21; no longer X11.A21
- net A25: now also X6.A22; no longer X11.A22
- net A26: now also X6.A23; no longer X11.A23
- net A27: now also X7.A27, X9.A27; no longer X1.A27, X5.A27
- net A28: now also X7.A28, X9.A28; no longer X1.A28, X5.A28
- net A29: now also X7.A29, X9.A29; no longer X1.A29, X5.A29
- net A30: now also X6.A27; no longer X11.A27
- net A31: now also X6.A28; no longer X11.A28
- net A32: now also X6.A29; no longer X11.A29
- net A39: now also X5.A17; no longer X21.A17
- net A40: now also X5.A18; no longer X21.A18
- net A41: now also X5.A19; no longer X21.A19
- net A42: now also X5.A20; no longer X21.A20
- net A43: now also X5.A21; no longer X21.A21
- net A44: now also X5.A22; no longer X21.A22
- net A45: now also X5.A23; no longer X21.A23
- net A46: now also X5.A27; no longer X21.A27
- net A47: now also X5.A28; no longer X21.A28
- net A48: now also X5.A29; no longer X21.A29
- net A5: now also X0.A5, X1_AUX.A5, X2.A5, X3_AUX.A5, X4.A5, X6.A5, X7.A5, X9.A5; no longer X1.A5
- net A71: now also X3_AUX.A17; no longer X7.A17
- net A72: now also X3_AUX.A18; no longer X7.A18
- net A73: now also X3_AUX.A19; no longer X7.A19
- net A74: now also X3_AUX.A20; no longer X7.A20
- net A75: now also X3_AUX.A21; no longer X7.A21
- net A76: now also X3_AUX.A22; no longer X7.A22
- net A77: now also X3_AUX.A23; no longer X7.A23
- net A78: now also X3_AUX.A27; no longer X7.A27
- net A79: now also X3_AUX.A28; no longer X7.A28
- net A8: now also X0.A8, X1_AUX.A8, X2.A8, X3_AUX.A8, X4.A8, X6.A8, X7.A8, X9.A8; no longer X1.A8
- net A80: now also X3_AUX.A29; no longer X7.A29
- net A87: now also X2.A17; no longer X8.A17
- net A88: now also X2.A18; no longer X8.A18
- net A89: now also X2.A19; no longer X8.A19
- net A9: now also X0.A9, X1_AUX.A9, X2.A9, X3_AUX.A9, X4.A9, X6.A9, X7.A9, X9.A9; no longer X1.A9
- net A90: now also X2.A20; no longer X8.A20
- net A91: now also X2.A21; no longer X8.A21
- net A92: now also X2.A22; no longer X8.A22
- net A93: now also X2.A23; no longer X8.A23
- net A94: now also X2.A27; no longer X8.A27
- net A95: now also X2.A28; no longer X8.A28
- net A96: now also X2.A29; no longer X8.A29
- net C103: now also X1_AUX.C17; no longer X9.C17
- net C104: now also X1_AUX.C18; no longer X9.C18
- net C105: now also X1_AUX.C19; no longer X9.C19
- net C106: now also X1_AUX.C20; no longer X9.C20
- net C107: now also X1_AUX.C21; no longer X9.C21
- net C108: now also X1_AUX.C22; no longer X9.C22
- net C109: now also X1_AUX.C23; no longer X9.C23
- net C11: now also X6.C17; no longer X11.C17
- net C110: now also X1_AUX.C27; no longer X9.C27
- net C111: now also X1_AUX.C28; no longer X9.C28
- net C112: now also X1_AUX.C29; no longer X9.C29
- net C119: now also X0.C17; no longer X10.C17
- net C12: now also X6.C18; no longer X11.C18
- net C120: now also X0.C18; no longer X10.C18
- net C121: now also X0.C19; no longer X10.C19
- net C122: now also X0.C20; no longer X10.C20
- net C123: now also X0.C21; no longer X10.C21
- net C124: now also X0.C22; no longer X10.C22
- net C125: now also X0.C23; no longer X10.C23
- net C126: now also X0.C27; no longer X10.C27
- net C127: now also X0.C28; no longer X10.C28
- net C128: now also X0.C29; no longer X10.C29
- net C13: now also X6.C19; no longer X11.C19
- net C14: now also X6.C20; no longer X11.C20
- net C15: now also X0.C15, X1_AUX.C15, X2.C15, X3_AUX.C15, X4.C15, X6.C15, X7.C15, X9.C15; no longer X1.C15
- net C16: now also X0.C16, X1_AUX.C16, X2.C16, X3_AUX.C16, X4.C16, X6.C16, X7.C16, X9.C16; no longer X1.C16
- net C17: now also X7.C17, X9.C17; no longer X1.C17, X5.C17
- net C18: now also X7.C18, X9.C18; no longer X1.C18, X5.C18
- net C19: now also X7.C19, X9.C19; no longer X1.C19, X5.C19
- net C2: now also X0.C2, X1_AUX.C2, X2.C2, X3_AUX.C2, X4.C2, X6.C2, X7.C2, X9.C2; no longer X1.C2
- net C20: now also X7.C20, X9.C20; no longer X1.C20, X5.C20
- net C21: now also X7.C21, X9.C21; no longer X1.C21, X5.C21
- net C22: now also X7.C22, X9.C22; no longer X1.C22, X5.C22
- net C23: now also X7.C23, X9.C23; no longer X1.C23, X5.C23
- net C24: now also X6.C21; no longer X11.C21
- net C25: now also X6.C22; no longer X11.C22
- net C26: now also X6.C23; no longer X11.C23
- net C27: now also X7.C27, X9.C27; no longer X1.C27, X5.C27
- net C28: now also X7.C28, X9.C28; no longer X1.C28, X5.C28
- net C29: now also X7.C29, X9.C29; no longer X1.C29, X5.C29
- net C30: now also X6.C27; no longer X11.C27
- net C31: now also X6.C28; no longer X11.C28
- net C32: now also X6.C29; no longer X11.C29
- net C39: now also X5.C17; no longer X21.C17
- net C40: now also X5.C18; no longer X21.C18
- net C41: now also X5.C19; no longer X21.C19
- net C42: now also X5.C20; no longer X21.C20
- net C43: now also X5.C21; no longer X21.C21
- net C44: now also X5.C22; no longer X21.C22
- net C45: now also X5.C23; no longer X21.C23
- net C46: now also X5.C27; no longer X21.C27
- net C47: now also X5.C28; no longer X21.C28
- net C48: now also X5.C29; no longer X21.C29
- net C5: now also X0.C5, X1_AUX.C5, X2.C5, X3_AUX.C5, X4.C5, X6.C5, X7.C5, X9.C5; no longer X1.C5
- net C71: now also X3_AUX.C17; no longer X7.C17
- net C72: now also X3_AUX.C18; no longer X7.C18
- net C73: now also X3_AUX.C19; no longer X7.C19
- net C74: now also X3_AUX.C20; no longer X7.C20
- net C75: now also X3_AUX.C21; no longer X7.C21
- net C76: now also X3_AUX.C22; no longer X7.C22
- net C77: now also X3_AUX.C23; no longer X7.C23
- net C78: now also X3_AUX.C27; no longer X7.C27
- net C79: now also X3_AUX.C28; no longer X7.C28
- net C8: now also X0.C8, X1_AUX.C8, X2.C8, X3_AUX.C8, X4.C8, X6.C8, X7.C8, X9.C8; no longer X1.C8
- net C80: now also X3_AUX.C29; no longer X7.C29
- net C87: now also X2.C17; no longer X8.C17
- net C88: now also X2.C18; no longer X8.C18
- net C89: now also X2.C19; no longer X8.C19
- net C9: now also X0.C9, X1_AUX.C9, X2.C9, X3_AUX.C9, X4.C9, X6.C9, X7.C9, X9.C9; no longer X1.C9
- net C90: now also X2.C20; no longer X8.C20
- net C91: now also X2.C21; no longer X8.C21
- net C92: now also X2.C22; no longer X8.C22
- net C93: now also X2.C23; no longer X8.C23
- net C94: now also X2.C27; no longer X8.C27
- net C95: now also X2.C28; no longer X8.C28
- net C96: now also X2.C29; no longer X8.C29
- net D0: now also X0.A10, X1_AUX.A10, X2.A10, X3_AUX.A10, X4.A10, X6.A10, X7.A10, X9.A10; no longer X1.A10
- net D1: now also X0.C10, X1_AUX.C10, X2.C10, X3_AUX.C10, X4.C10, X6.C10, X7.C10, X9.C10; no longer X1.C10
- net D2: now also X0.A11, X1_AUX.A11, X2.A11, X3_AUX.A11, X4.A11, X6.A11, X7.A11, X9.A11; no longer X1.A11
- net D3: now also X0.C11, X1_AUX.C11, X2.C11, X3_AUX.C11, X4.C11, X6.C11, X7.C11, X9.C11; no longer X1.C11
- net GND: now also X0.A1, X0.C1, X1_AUX.A1, X1_AUX.C1, X2.A1, X2.C1, X3_AUX.A1, X3_AUX.C1, X4.A1, X4.C1, X6.A1, X6.C1, X7.A1, X7.A25, X7.C1, X7.C25, X9.A1, X9.A25, X9.C1, X9.C25; no longer X1.A1, X1.A25, X1.C1, X1.C25, X11.A1, X5.A25, X5.C25
- net GND1: now also X6.A25, X6.C25; no longer X11.A25, X11.C1, X11.C25
- net GND2: now also X5.A25, X5.C25; no longer X21.A1, X21.A25, X21.C1, X21.C25
- net GND3: no longer X4.A1, X4.C1
- net GND4: now also X3_AUX.A25, X3_AUX.C25; no longer X7.A1, X7.A25, X7.C1, X7.C25
- net GND5: now also X2.A25, X2.C25; no longer X8.A1, X8.A25, X8.C1, X8.C25
- net GND6: now also X1_AUX.A25, X1_AUX.C25; no longer X9.A1, X9.A25, X9.C1, X9.C25
- net GND7: now also X0.A25, X0.C25; no longer X10.A1, X10.A25, X10.C1, X10.C25
- net GPIO0: now also X0.A3, X1_AUX.A3, X2.A3, X3_AUX.A3, X4.A3, X6.A3, X7.A3, X9.A3; no longer X1.A3
- net GPIO1: now also X0.C3, X1_AUX.C3, X2.C3, X3_AUX.C3, X4.C3, X6.C3, X7.C3, X9.C3; no longer X1.C3
- net GPIO2: now also X1_AUX.A4, X2.A4, X3_AUX.A4, X4.A4, X6.A4, X7.A4, X9.A4; no longer X1.A4
- net GPIO3: now also X1_AUX.C4, X2.C4, X3_AUX.C4, X4.C4, X6.C4, X7.C4, X9.C4; no longer X1.C4
- net GPIO4: now also X0.A6, X1_AUX.A6, X2.A6, X3_AUX.A6, X4.A6, X6.A6, X7.A6, X9.A6; no longer X1.A6
- net GPIO5: now also X0.C6, X1_AUX.C6, X2.C6, X3_AUX.C6, X4.C6, X6.C6, X7.C6, X9.C6; no longer X1.C6
- net GPIO57: now also X0.A4; no longer X10.A4
- net GPIO6: now also X0.A7, X1_AUX.A7, X2.A7, X3_AUX.A7, X4.A7, X6.A7, X7.A7, X9.A7; no longer X1.A7
- net GPIO61: now also X0.C4; no longer X10.C4
- net GPIO7: now also X0.C7, X1_AUX.C7, X2.C7, X3_AUX.C7, X4.C7, X6.C7, X7.C7, X9.C7; no longer X1.C7
- net HV: now also X7.A26, X7.C26, X9.A26, X9.C26; no longer X1.A26, X1.C26, X5.A26, X5.C26
- net HV1: now also X6.A26, X6.C26; no longer X11.A26, X11.C26
- net HV2: now also X5.A26, X5.C26; no longer X21.A26, X21.C26
- net HV4: now also X3_AUX.A26, X3_AUX.C26; no longer X7.A26, X7.C26
- net HV5: now also X2.A26, X2.C26; no longer X8.A26, X8.C26
- net HV6: now also X1_AUX.A26, X1_AUX.C26; no longer X9.A26, X9.C26
- net HV7: now also X0.A26, X0.C26; no longer X10.A26, X10.C26
- net HV_INTERLOCK: now also X7.A24, X7.C24, X9.A24, X9.C24; no longer X1.A24, X1.C24, X5.A24, X5.C24
- net HV_INTERLOCK1: now also X6.A24, X6.C24; no longer X11.A24, X11.C24
- net HV_INTERLOCK2: now also X5.A24, X5.C24; no longer X21.A24, X21.C24
- net HV_INTERLOCK4: now also X3_AUX.A24, X3_AUX.C24; no longer X7.A24, X7.C24
- net HV_INTERLOCK5: now also X2.A24, X2.C24; no longer X8.A24, X8.C24
- net HV_INTERLOCK6: now also X1_AUX.A24, X1_AUX.C24; no longer X9.A24, X9.C24
- net HV_INTERLOCK7: now also X0.A24, X0.C24; no longer X10.A24, X10.C24
- net I2C_SCL: now also X0.C14, X1_AUX.C14, X2.C14, X3_AUX.C14, X4.C14, X6.C14, X7.C14, X9.C14; no longer X1.C14
- net I2C_SDA: now also X0.A14, X1_AUX.A14, X2.A14, X3_AUX.A14, X4.A14, X6.A14, X7.A14, X9.A14; no longer X1.A14
- net SPI_CS2: now also TEENSY.26, X2.C12; no longer TEENSY.29
- net SPI_CS4: now also TEENSY.28, X4.C12; no longer TEENSY.31
- net SPI_CS5: now also TEENSY.29; no longer TEENSY.32, X10.C12, X11.C12, X21.C12, X4.C12, X7.C12, X8.C12, X9.C12
- net SPI_CS6: now also TEENSY.30, X6.C12; no longer TEENSY.33, X1.C12
- net SPI_MISO: now also X0.C13, X1_AUX.C13, X2.C13, X3_AUX.C13, X4.C13, X6.C13, X7.C13, X9.C13; no longer X1.C13
- net SPI_MOSI: now also X0.A13, X1_AUX.A13, X2.A13, X3_AUX.A13, X4.A13, X6.A13, X7.A13, X9.A13; no longer X1.A13
- net SPI_SCLK: now also X0.A12, X1_AUX.A12, X2.A12, X3_AUX.A12, X4.A12, X6.A12, X7.A12, X9.A12; no longer X1.A12
- net VREF: now also X7.A32, X7.C32, X9.A32, X9.C32; no longer X1.A32, X1.C32, X5.A32, X5.C32
- net VREF1: now also X6.A32, X6.C32; no longer X11.A32, X11.C32
- net VREF2: now also X5.A32, X5.C32; no longer X21.A32, X21.C32
- net VREF4: now also X3_AUX.A32, X3_AUX.C32; no longer X7.A32, X7.C32
- net VREF5: now also X2.A32, X2.C32; no longer X8.A32, X8.C32
- net VREF6: now also X1_AUX.A32, X1_AUX.C32; no longer X9.A32, X9.C32
- net VREF7: now also X0.A32, X0.C32; no longer X10.A32, X10.C32
Routing:
- net SPI_CS7: track 0.00 -> 134.8 mm
- net SPI_CS7_AUX: track 79.6 -> 0.00 mm
- net SPI_CS8_AUX: track 0.00 -> 77.8 mm
- net SPI_CS5: track 99.0 -> 40.4 mm
- net SPI_CS3_AUX: track 0.00 -> 52.3 mm
- net SPI_C0: track 52.3 -> 0.00 mm
- net SPI_CS1: track 44.0 -> 0.00 mm
- net SPI_CS3: track 40.4 -> 0.00 mm
- net SPI_CS2: track 40.4 -> 0.00 mm
- net SPI_CS9: track 0.00 -> 25.9 mm
- net SPI_CS6: track 31.3 -> 40.4 mm
- net SPI_CS4: track 41.1 -> 44.0 mm

Commit message: Incremental progress
Parts:
- added JP1: (no value), pinhead:1X02
Connections:
- removed net +15V1: X6.A31, X6.C31
- removed net +15V2: X5.A31, X5.C31
- removed net +15V3: X4.A31, X4.C31
- removed net +15V4: X3_AUX.A31, X3_AUX.C31
- removed net +15V5: X2.A31, X2.C31
- removed net +15V6: X1_AUX.A31, X1_AUX.C31
- removed net +15V7: X0.A31, X0.C31
- removed net -15V1: X6.A30, X6.C30
- removed net -15V2: X5.A30, X5.C30
- removed net -15V3: X4.A30, X4.C30
- removed net -15V4: X3_AUX.A30, X3_AUX.C30
- removed net -15V5: X2.A30, X2.C30
- removed net -15V6: X1_AUX.A30, X1_AUX.C30
- removed net -15V7: X0.A30, X0.C30
- removed net A103: X1_AUX.A17
- removed net A104: X1_AUX.A18
- removed net A105: X1_AUX.A19
- removed net A106: X1_AUX.A20
- removed net A107: X1_AUX.A21
- removed net A108: X1_AUX.A22
- removed net A109: X1_AUX.A23
- removed net A11: X6.A17
- removed net A110: X1_AUX.A27
- removed net A111: X1_AUX.A28
- removed net A112: X1_AUX.A29
- removed net A119: X0.A17
- removed net A12: X6.A18
- removed net A120: X0.A18
- removed net A121: X0.A19
- removed net A122: X0.A20
- removed net A123: X0.A21
- removed net A124: X0.A22
- removed net A125: X0.A23
- removed net A126: X0.A27
- removed net A127: X0.A28
- removed net A128: X0.A29
- removed net A13: X6.A19
- removed net A14: X6.A20
- removed net A24: X6.A21
- removed net A25: X6.A22
- removed net A26: X6.A23
- removed net A30: X6.A27
- removed net A31: X6.A28
- removed net A32: X6.A29
- removed net A39: X5.A17
- removed net A40: X5.A18
- removed net A41: X5.A19
- removed net A42: X5.A20
- removed net A43: X5.A21
- removed net A44: X5.A22
- removed net A45: X5.A23
- removed net A46: X5.A27
- removed net A47: X5.A28
- removed net A48: X5.A29
- removed net A55: X4.A17
- removed net A56: X4.A18
- removed net A57: X4.A19
- removed net A58: X4.A20
- removed net A59: X4.A21
- removed net A60: X4.A22
- removed net A61: X4.A23
- removed net A62: X4.A27
- removed net A63: X4.A28
- removed net A64: X4.A29
- removed net A71: X3_AUX.A17
- removed net A72: X3_AUX.A18
- removed net A73: X3_AUX.A19
- removed net A74: X3_AUX.A20
- removed net A75: X3_AUX.A21
- removed net A76: X3_AUX.A22
- removed net A77: X3_AUX.A23
- removed net A78: X3_AUX.A27
- removed net A79: X3_AUX.A28
- removed net A80: X3_AUX.A29
- removed net A87: X2.A17
- removed net A88: X2.A18
- removed net A89: X2.A19
- removed net A90: X2.A20
- removed net A91: X2.A21
- removed net A92: X2.A22
- removed net A93: X2.A23
- removed net A94: X2.A27
- removed net A95: X2.A28
- removed net A96: X2.A29
- removed net C103: X1_AUX.C17
- removed net C104: X1_AUX.C18
- removed net C105: X1_AUX.C19
- removed net C106: X1_AUX.C20
- removed net C107: X1_AUX.C21
- removed net C108: X1_AUX.C22
- removed net C109: X1_AUX.C23
- removed net C11: X6.C17
- removed net C110: X1_AUX.C27
- removed net C111: X1_AUX.C28
- removed net C112: X1_AUX.C29
- removed net C119: X0.C17
- removed net C12: X6.C18
- removed net C120: X0.C18
- removed net C121: X0.C19
- removed net C122: X0.C20
- removed net C123: X0.C21
- removed net C124: X0.C22
- removed net C125: X0.C23
- removed net C126: X0.C27
- removed net C127: X0.C28
- removed net C128: X0.C29
- removed net C13: X6.C19
- removed net C14: X6.C20
- removed net C24: X6.C21
- removed net C25: X6.C22
- removed net C26: X6.C23
- removed net C30: X6.C27
- removed net C31: X6.C28
- removed net C32: X6.C29
- removed net C39: X5.C17
- removed net C40: X5.C18
- removed net C41: X5.C19
- removed net C42: X5.C20
- removed net C43: X5.C21
- removed net C44: X5.C22
- removed net C45: X5.C23
- removed net C46: X5.C27
- removed net C47: X5.C28
- removed net C48: X5.C29
- removed net C55: X4.C17
- removed net C56: X4.C18
- removed net C57: X4.C19
- removed net C58: X4.C20
- removed net C59: X4.C21
- removed net C60: X4.C22
- removed net C61: X4.C23
- removed net C62: X4.C27
- removed net C63: X4.C28
- removed net C64: X4.C29
- removed net C71: X3_AUX.C17
- removed net C72: X3_AUX.C18
- removed net C73: X3_AUX.C19
- removed net C74: X3_AUX.C20
- removed net C75: X3_AUX.C21
- removed net C76: X3_AUX.C22
- removed net C77: X3_AUX.C23
- removed net C78: X3_AUX.C27
- removed net C79: X3_AUX.C28
- removed net C80: X3_AUX.C29
- removed net C87: X2.C17
- removed net C88: X2.C18
- removed net C89: X2.C19
- removed net C90: X2.C20
- removed net C91: X2.C21
- removed net C92: X2.C22
- removed net C93: X2.C23
- removed net C94: X2.C27
- removed net C95: X2.C28
- removed net C96: X2.C29
- removed net GND1: X6.A25, X6.C25
- removed net GND2: X5.A25, X5.C25
- removed net GND3: X4.A25, X4.C25
- removed net GND4: X3_AUX.A25, X3_AUX.C25
- removed net GND5: X2.A25, X2.C25
- removed net GND6: X1_AUX.A25, X1_AUX.C25
- removed net GND7: X0.A25, X0.C25
- removed net GPIO57: X0.A4
- removed net GPIO61: X0.C4
- removed net HV1: X6.A26, X6.C26
- removed net HV2: X5.A26, X5.C26
- removed net HV3: X4.A26, X4.C26
- removed net HV4: X3_AUX.A26, X3_AUX.C26
- removed net HV5: X2.A26, X2.C26
- removed net HV6: X1_AUX.A26, X1_AUX.C26
- removed net HV7: X0.A26, X0.C26
- removed net HV_INTERLOCK1: X6.A24, X6.C24
- removed net HV_INTERLOCK2: X5.A24, X5.C24
- removed net HV_INTERLOCK3: X4.A24, X4.C24
- removed net HV_INTERLOCK4: X3_AUX.A24, X3_AUX.C24
- removed net HV_INTERLOCK5: X2.A24, X2.C24
- removed net HV_INTERLOCK6: X1_AUX.A24, X1_AUX.C24
- removed net HV_INTERLOCK7: X0.A24, X0.C24
- removed net VREF1: X6.A32, X6.C32
- removed net VREF2: X5.A32, X5.C32
- removed net VREF3: X4.A32, X4.C32
- removed net VREF4: X3_AUX.A32, X3_AUX.C32
- removed net VREF5: X2.A32, X2.C32
- removed net VREF6: X1_AUX.A32, X1_AUX.C32
- removed net VREF7: X0.A32, X0.C32
- net +15V: now also X0.A31, X0.C31, X1_AUX.A31, X1_AUX.C31, X2.A31, X2.C31, X3_AUX.A31, X3_AUX.C31, X4.A31, X4.C31, X5.A31, X5.C31, X6.A31, X6.C31
- net -15V: now also X0.A30, X0.C30, X1_AUX.A30, X1_AUX.C30, X2.A30, X2.C30, X3_AUX.A30, X3_AUX.C30, X4.A30, X4.C30, X5.A30, X5.C30, X6.A30, X6.C30
- net A17: now also X0.A17, X1_AUX.A17, X2.A17, X3_AUX.A17, X4.A17, X5.A17, X6.A17
- net A18: now also X0.A18, X1_AUX.A18, X2.A18, X3_AUX.A18, X4.A18, X5.A18, X6.A18
- net A19: now also X0.A19, X1_AUX.A19, X2.A19, X3_AUX.A19, X4.A19, X5.A19, X6.A19
- net A20: now also X0.A20, X1_AUX.A20, X2.A20, X3_AUX.A20, X4.A20, X5.A20, X6.A20
- net A21: now also X0.A21, X1_AUX.A21, X2.A21, X3_AUX.A21, X4.A21, X5.A21, X6.A21
- net A22: now also X0.A22, X1_AUX.A22, X2.A22, X3_AUX.A22, X4.A22, X5.A22, X6.A22
- net A23: now also X0.A23, X1_AUX.A23, X2.A23, X3_AUX.A23, X4.A23, X5.A23, X6.A23
- net A27: now also X0.A27, X1_AUX.A27, X2.A27, X3_AUX.A27, X4.A27, X5.A27, X6.A27
- net A28: now also X0.A28, X1_AUX.A28, X2.A28, X3_AUX.A28, X4.A28, X5.A28, X6.A28
- net A29: now also X0.A29, X1_AUX.A29, X2.A29, X3_AUX.A29, X4.A29, X5.A29, X6.A29
- net C17: now also X0.C17, X1_AUX.C17, X2.C17, X3_AUX.C17, X4.C17, X5.C17, X6.C17
- net C18: now also X0.C18, X1_AUX.C18, X2.C18, X3_AUX.C18, X4.C18, X5.C18, X6.C18
- net C19: now also X0.C19, X1_AUX.C19, X2.C19, X3_AUX.C19, X4.C19, X5.C19, X6.C19
- net C20: now also X0.C20, X1_AUX.C20, X2.C20, X3_AUX.C20, X4.C20, X5.C20, X6.C20
- net C21: now also X0.C21, X1_AUX.C21, X2.C21, X3_AUX.C21, X4.C21, X5.C21, X6.C21
- net C22: now also X0.C22, X1_AUX.C22, X2.C22, X3_AUX.C22, X4.C22, X5.C22, X6.C22
- net C23: now also X0.C23, X1_AUX.C23, X2.C23, X3_AUX.C23, X4.C23, X5.C23, X6.C23
- net C27: now also X0.C27, X1_AUX.C27, X2.C27, X3_AUX.C27, X4.C27, X5.C27, X6.C27
- net C28: now also X0.C28, X1_AUX.C28, X2.C28, X3_AUX.C28, X4.C28, X5.C28, X6.C28
- net C29: now also X0.C29, X1_AUX.C29, X2.C29, X3_AUX.C29, X4.C29, X5.C29, X6.C29
- net GND: now also JP1.2, X0.A25, X0.C25, X1_AUX.A25, X1_AUX.C25, X2.A25, X2.C25, X3_AUX.A25, X3_AUX.C25, X4.A25, X4.C25, X5.A25, X5.C25, X6.A25, X6.C25
- net GPIO2: now also X0.A4
- net GPIO3: now also X0.C4
- net HV: now also JP1.1, X0.A26, X0.C26, X1_AUX.A26, X1_AUX.C26, X2.A26, X2.C26, X3_AUX.A26, X3_AUX.C26, X4.A26, X4.C26, X5.A26, X5.C26, X6.A26, X6.C26
- net HV_INTERLOCK: now also X0.A24, X0.C24, X1_AUX.A24, X1_AUX.C24, X2.A24, X2.C24, X3_AUX.A24, X3_AUX.C24, X4.A24, X4.C24, X5.A24, X5.C24, X6.A24, X6.C24
- net VREF: now also X0.A32, X0.C32, X1_AUX.A32, X1_AUX.C32, X2.A32, X2.C32, X3_AUX.A32, X3_AUX.C32, X4.A32, X4.C32, X5.A32, X5.C32, X6.A32, X6.C32
Other:
- board text added: "HV!"
- board text added: "High Voltage!"

Commit message: Version 1.0 board layout pretty much done
Parts:
- removed X0, X1_AUX, X3_AUX, X9: FAC64S, Eurocard-Backplane-jqi:FAC64S
- added X1, X10_AUX, X9_AUX: FAC64S, Eurocard-Backplane-jqi:FAC64S
- added X11: (no value), Eurocard-Backplane-jqi:5566-4
- X3: value (none) -> FAC64S; device Eurocard-Backplane-jqi:5566-4 -> Eurocard-Backplane-jqi:FAC64S
- moved X8_AUX 304.8 mm to (48.3, 64.8), flipped to the top
- moved X3 275.2 mm to (139.7, 64.8), flipped to the top, turned to 0 degrees
- moved X7 61.0 mm to (383.5, 64.8)
- moved X4 61.0 mm to (200.7, 64.8)
- moved X5 61.0 mm to (261.6, 64.8)
- moved X6 61.0 mm to (322.6, 64.8)
- moved X2 0.13 mm to (78.7, 64.8)
- moved C2 0.13 mm to (368.3, 16.4)
- moved C3 0.13 mm to (337.8, 16.4)
- moved C5 0.13 mm to (403.6, 39.0)
- moved J1 0.13 mm to (419.1, 26.5)
- moved U2 0.13 mm to (410.2, 53.2)
- moved U$3 0.13 mm to (0.00, -0.13)
- moved L1 0.13 mm to (421.6, 31.6)
- moved C1 0.13 mm to (415.5, 112.6)
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Connections:
- removed net SPI_CS0: TEENSY.24, X0.C12
- removed net SPI_CS1_AUX: TEENSY.25, X1_AUX.C12
- removed net SPI_CS3_AUX: TEENSY.27, X3_AUX.C12
- removed net SPI_CS9: TEENSY.33, X9.C12
- new net SPI_CS1: TEENSY.24, X1.C12
- new net SPI_CS10_AUX: TEENSY.32, X10_AUX.C12
- new net SPI_CS3: TEENSY.28, X3.C12
- new net SPI_CS9_AUX: TEENSY.27, X9_AUX.C12
- net +15V: now also X1.A31, X1.C31, X10_AUX.A31, X10_AUX.C31, X11.2, X3.A31, X3.C31, X9_AUX.A31, X9_AUX.C31; no longer X0.A31, X0.C31, X1_AUX.A31, X1_AUX.C31, X3.2, X3_AUX.A31, X3_AUX.C31, X9.A31, X9.C31
- net -15V: now also X1.A30, X1.C30, X10_AUX.A30, X10_AUX.C30, X11.1, X3.A30, X3.C30, X9_AUX.A30, X9_AUX.C30; no longer X0.A30, X0.C30, X1_AUX.A30, X1_AUX.C30, X3.1, X3_AUX.A30, X3_AUX.C30, X9.A30, X9.C30
- net A15: now also X1.A15, X10_AUX.A15, X3.A15, X9_AUX.A15; no longer X0.A15, X1_AUX.A15, X3_AUX.A15, X9.A15
- net A16: now also X1.A16, X10_AUX.A16, X3.A16, X9_AUX.A16; no longer X0.A16, X1_AUX.A16, X3_AUX.A16, X9.A16
- net A17: now also X1.A17, X10_AUX.A17, X3.A17, X9_AUX.A17; no longer X0.A17, X1_AUX.A17, X3_AUX.A17, X9.A17
- net A18: now also X1.A18, X10_AUX.A18, X3.A18, X9_AUX.A18; no longer X0.A18, X1_AUX.A18, X3_AUX.A18, X9.A18
- net A19: now also X1.A19, X10_AUX.A19, X3.A19, X9_AUX.A19; no longer X0.A19, X1_AUX.A19, X3_AUX.A19, X9.A19
- net A2: now also X1.A2, X10_AUX.A2, X3.A2, X9_AUX.A2; no longer X0.A2, X1_AUX.A2, X3_AUX.A2, X9.A2
- net A20: now also X1.A20, X10_AUX.A20, X3.A20, X9_AUX.A20; no longer X0.A20, X1_AUX.A20, X3_AUX.A20, X9.A20
- net A21: now also X1.A21, X10_AUX.A21, X3.A21, X9_AUX.A21; no longer X0.A21, X1_AUX.A21, X3_AUX.A21, X9.A21
- net A22: now also X1.A22, X10_AUX.A22, X3.A22, X9_AUX.A22; no longer X0.A22, X1_AUX.A22, X3_AUX.A22, X9.A22
- net A23: now also X1.A23, X10_AUX.A23, X3.A23, X9_AUX.A23; no longer X0.A23, X1_AUX.A23, X3_AUX.A23, X9.A23
- net A27: now also X1.A27, X10_AUX.A27, X3.A27, X9_AUX.A27; no longer X0.A27, X1_AUX.A27, X3_AUX.A27, X9.A27
- net A28: now also X1.A28, X10_AUX.A28, X3.A28, X9_AUX.A28; no longer X0.A28, X1_AUX.A28, X3_AUX.A28, X9.A28
- net A29: now also X1.A29, X10_AUX.A29, X3.A29, X9_AUX.A29; no longer X0.A29, X1_AUX.A29, X3_AUX.A29, X9.A29
- net A5: now also X1.A5, X10_AUX.A5, X3.A5, X9_AUX.A5; no longer X0.A5, X1_AUX.A5, X3_AUX.A5, X9.A5
- net A8: now also X1.A8, X10_AUX.A8, X3.A8, X9_AUX.A8; no longer X0.A8, X1_AUX.A8, X3_AUX.A8, X9.A8
- net A9: now also X1.A9, X10_AUX.A9, X3.A9, X9_AUX.A9; no longer X0.A9, X1_AUX.A9, X3_AUX.A9, X9.A9
- net C15: now also X1.C15, X10_AUX.C15, X3.C15, X9_AUX.C15; no longer X0.C15, X1_AUX.C15, X3_AUX.C15, X9.C15
- net C16: now also X1.C16, X10_AUX.C16, X3.C16, X9_AUX.C16; no longer X0.C16, X1_AUX.C16, X3_AUX.C16, X9.C16
- net C17: now also X1.C17, X10_AUX.C17, X3.C17, X9_AUX.C17; no longer X0.C17, X1_AUX.C17, X3_AUX.C17, X9.C17
- net C18: now also X1.C18, X10_AUX.C18, X3.C18, X9_AUX.C18; no longer X0.C18, X1_AUX.C18, X3_AUX.C18, X9.C18
- net C19: now also X1.C19, X10_AUX.C19, X3.C19, X9_AUX.C19; no longer X0.C19, X1_AUX.C19, X3_AUX.C19, X9.C19
- net C2: now also X1.C2, X10_AUX.C2, X3.C2, X9_AUX.C2; no longer X0.C2, X1_AUX.C2, X3_AUX.C2, X9.C2
- net C20: now also X1.C20, X10_AUX.C20, X3.C20, X9_AUX.C20; no longer X0.C20, X1_AUX.C20, X3_AUX.C20, X9.C20
- net C21: now also X1.C21, X10_AUX.C21, X3.C21, X9_AUX.C21; no longer X0.C21, X1_AUX.C21, X3_AUX.C21, X9.C21
- net C22: now also X1.C22, X10_AUX.C22, X3.C22, X9_AUX.C22; no longer X0.C22, X1_AUX.C22, X3_AUX.C22, X9.C22
- net C23: now also X1.C23, X10_AUX.C23, X3.C23, X9_AUX.C23; no longer X0.C23, X1_AUX.C23, X3_AUX.C23, X9.C23
- net C27: now also X1.C27, X10_AUX.C27, X3.C27, X9_AUX.C27; no longer X0.C27, X1_AUX.C27, X3_AUX.C27, X9.C27
- net C28: now also X1.C28, X10_AUX.C28, X3.C28, X9_AUX.C28; no longer X0.C28, X1_AUX.C28, X3_AUX.C28, X9.C28
- net C29: now also X1.C29, X10_AUX.C29, X3.C29, X9_AUX.C29; no longer X0.C29, X1_AUX.C29, X3_AUX.C29, X9.C29
- net C5: now also X1.C5, X10_AUX.C5, X3.C5, X9_AUX.C5; no longer X0.C5, X1_AUX.C5, X3_AUX.C5, X9.C5
- net C8: now also X1.C8, X10_AUX.C8, X3.C8, X9_AUX.C8; no longer X0.C8, X1_AUX.C8, X3_AUX.C8, X9.C8
- net C9: now also X1.C9, X10_AUX.C9, X3.C9, X9_AUX.C9; no longer X0.C9, X1_AUX.C9, X3_AUX.C9, X9.C9
- net D0: now also X1.A10, X10_AUX.A10, X3.A10, X9_AUX.A10; no longer X0.A10, X1_AUX.A10, X3_AUX.A10, X9.A10
- net D1: now also X1.C10, X10_AUX.C10, X3.C10, X9_AUX.C10; no longer X0.C10, X1_AUX.C10, X3_AUX.C10, X9.C10
- net D2: now also X1.A11, X10_AUX.A11, X3.A11, X9_AUX.A11; no longer X0.A11, X1_AUX.A11, X3_AUX.A11, X9.A11
- net D3: now also X1.C11, X10_AUX.C11, X3.C11, X9_AUX.C11; no longer X0.C11, X1_AUX.C11, X3_AUX.C11, X9.C11
- net GND: now also X1.A1, X1.A25, X1.C1, X1.C25, X10_AUX.A1, X10_AUX.A25, X10_AUX.C1, X10_AUX.C25, X11.3, X11.4, X3.A1, X3.A25, X3.C1, X3.C25, X9_AUX.A1, X9_AUX.A25, X9_AUX.C1, X9_AUX.C25; no longer X0.A1, X0.A25, X0.C1, X0.C25, X1_AUX.A1, X1_AUX.A25, X1_AUX.C1, X1_AUX.C25, X3.3, X3.4, X3_AUX.A1, X3_AUX.A25, X3_AUX.C1, X3_AUX.C25, X9.A1, X9.A25, X9.C1, X9.C25
- net GPIO0: now also X1.A3, X10_AUX.A3, X3.A3, X9_AUX.A3; no longer X0.A3, X1_AUX.A3, X3_AUX.A3, X9.A3
- net GPIO1: now also X1.C3, X10_AUX.C3, X3.C3, X9_AUX.C3; no longer X0.C3, X1_AUX.C3, X3_AUX.C3, X9.C3
- net GPIO2: now also X1.A4, X10_AUX.A4, X3.A4, X9_AUX.A4; no longer X0.A4, X1_AUX.A4, X3_AUX.A4, X9.A4
- net GPIO3: now also X1.C4, X10_AUX.C4, X3.C4, X9_AUX.C4; no longer X0.C4, X1_AUX.C4, X3_AUX.C4, X9.C4
- net GPIO4: now also X1.A6, X10_AUX.A6, X3.A6, X9_AUX.A6; no longer X0.A6, X1_AUX.A6, X3_AUX.A6, X9.A6
- net GPIO5: now also X1.C6, X10_AUX.C6, X3.C6, X9_AUX.C6; no longer X0.C6, X1_AUX.C6, X3_AUX.C6, X9.C6
- net GPIO6: now also X1.A7, X10_AUX.A7, X3.A7, X9_AUX.A7; no longer X0.A7, X1_AUX.A7, X3_AUX.A7, X9.A7
- net GPIO7: now also X1.C7, X10_AUX.C7, X3.C7, X9_AUX.C7; no longer X0.C7, X1_AUX.C7, X3_AUX.C7, X9.C7
- net HV: now also X1.A26, X1.C26, X10_AUX.A26, X10_AUX.C26, X3.A26, X3.C26, X9_AUX.A26, X9_AUX.C26; no longer X0.A26, X0.C26, X1_AUX.A26, X1_AUX.C26, X3_AUX.A26, X3_AUX.C26, X9.A26, X9.C26
- net HV_INTERLOCK: now also X1.A24, X1.C24, X10_AUX.A24, X10_AUX.C24, X3.A24, X3.C24, X9_AUX.A24, X9_AUX.C24; no longer X0.A24, X0.C24, X1_AUX.A24, X1_AUX.C24, X3_AUX.A24, X3_AUX.C24, X9.A24, X9.C24
- net I2C_SCL: now also X1.C14, X10_AUX.C14, X3.C14, X9_AUX.C14; no longer X0.C14, X1_AUX.C14, X3_AUX.C14, X9.C14
- net I2C_SDA: now also X1.A14, X10_AUX.A14, X3.A14, X9_AUX.A14; no longer X0.A14, X1_AUX.A14, X3_AUX.A14, X9.A14
- net SPI_CS4: now also TEENSY.29; no longer TEENSY.28
- net SPI_CS5: now also TEENSY.30; no longer TEENSY.29
- net SPI_CS6: now also TEENSY.31; no longer TEENSY.30
- net SPI_CS7: now also TEENSY.33; no longer TEENSY.31
- net SPI_CS8_AUX: now also TEENSY.25; no longer TEENSY.32
- net SPI_MISO: now also X1.C13, X10_AUX.C13, X3.C13, X9_AUX.C13; no longer X0.C13, X1_AUX.C13, X3_AUX.C13, X9.C13
- net SPI_MOSI: now also X1.A13, X10_AUX.A13, X3.A13, X9_AUX.A13; no longer X0.A13, X1_AUX.A13, X3_AUX.A13, X9.A13
- net SPI_SCLK: now also X1.A12, X10_AUX.A12, X3.A12, X9_AUX.A12; no longer X0.A12, X1_AUX.A12, X3_AUX.A12, X9.A12
- net VREF: now also X1.A32, X1.C32, X10_AUX.A32, X10_AUX.C32, X3.A32, X3.C32, X9_AUX.A32, X9_AUX.C32; no longer X0.A32, X0.C32, X1_AUX.A32, X1_AUX.C32, X3_AUX.A32, X3_AUX.C32, X9.A32, X9.C32
Routing:
- net SPI_CS1: track 0.00 -> 453.3 mm
- net SPI_CS2: track 0.00 -> 367.0 mm
- net SPI_CS9_AUX: track 0.00 -> 328.3 mm
- net SPI_CS8_AUX: track 77.8 -> 405.8 mm
- net SPI_MOSI: track 121.4 -> 444.3 mm
- net SPI_SCLK: track 98.3 -> 410.6 mm
- net GPIO0: track 75.2 -> 387.3 mm
- net SPI_MISO: track 128.5 -> 440.6 mm
- net A29: track 62.4 -> 374.3 mm
- net A21: track 62.4 -> 374.3 mm
- net A28: track 62.4 -> 374.3 mm
- net A8: track 62.3 -> 374.2 mm
- net C27: track 62.3 -> 374.2 mm
- net D0: track 113.6 -> 425.5 mm
- net A27: track 62.3 -> 374.2 mm
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Other:
- board text added: "MOD1"
- board text added: "MOD10_AUX"
- board text added: "MOD2"
- board text added: "MOD3"
- board text added: "MOD4"
- board text added: "MOD7"
- board text added: "MOD8_AUX"
- board text added: "MOD9_AUX"
- board text added: "v1.0"
- board text removed: "MOD7_AUX"
- board text removed: "Test board - v0.1"
