File: EurocardBackplane.brd (EAGLE design)
At the start: 426.7 x 129.8 mm, 59 parts, among them U1 TXB0108, U2 TXB0108, U3 TXB0108, U4 TXB0108, U5 TXB0108, U6 TXB0108, U7 TXB0108, X1 FAC64S, X2 FAC64S, X3 FAC64S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

Commit message: adding just few traces
Routing:
- net A10: track 0.00 -> 30.3 mm
- net A3: track 372.1 -> 398.5 mm
- net A11: track 0.00 -> 24.1 mm
- net C10: track 0.00 -> 23.4 mm
- net C11: track 0.00 -> 17.4 mm
Changed lines of the file:
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@@
 <?xml version="1.0" encoding="utf-8"?>
 <!DOCTYPE eagle SYSTEM "eagle.dtd">
-<eagle version="6.6.0">
+<eagle version="7.7.0">
 <drawing>
 <settings>
@@
 <layer number="60" name="bCarbon" color="7" fill="1" visible="no" active="no"/>
 <layer number="61" name="stand" color="7" fill="1" visible="no" active="no"/>
-<layer number="90" name="Modules" color="7" fill="1" visible="no" active="yes"/>
+<layer number="90" name="Modules" color="7" fill="1" visible="no" active="no"/>
 <layer number="91" name="Nets" color="2" fill="1" visible="no" active="no"/>
 <layer number="92" name="Busses" color="1" fill="1" visible="no" active="no"/>
@@
 <pass name="Default">
 <param name="RoutingGrid" value="50mil"/>
+<param name="AutoGrid" value="1"/>
+<param name="Efforts" value="0"/>
+<param name="TopRouterVariant" value="1"/>
 <param name="tpViaShape" value="round"/>
 <param name="PrefDir.1" value="|"/>
@@
 <contactref element="U7" pad="12"/>
 <contactref element="X9" pad="A2"/>
+<wire x1="396.4268" y1="81.365" x2="397.087" y2="81.365" width="0.3048" layer="16"/>
+<wire x1="397.087" y1="81.365" x2="397.764" y2="82.042" width="0.3048" layer="16"/>
+<wire x1="397.764" y1="82.042" x2="397.764" y2="100.584" width="0.3048" layer="16"/>
+<wire x1="397.764" y1="100.584" x2="400.05" y2="102.87" width="0.3048" layer="16"/>
+<wire x1="400.05" y1="102.87" x2="405.13" y2="102.87" width="0.3048" layer="16"/>
+<wire x1="405.13" y1="102.87" x2="406.4" y2="101.6" width="0.3048" layer="16"/>
 <wire x1="91.6268" y1="81.365" x2="152.5868" y2="81.365" width="0" layer="19" extent="16-16"/>
 <wire x1="30.6668" y1="81.365" x2="91.6268" y2="81.365" width="0" layer="19" extent="16-16"/>
@@
 <wire x1="335.4668" y1="81.365" x2="274.5068" y2="81.365" width="0" layer="19" extent="16-16"/>
 <wire x1="396.4268" y1="81.365" x2="335.4668" y2="81.365" width="0" layer="19" extent="16-16"/>
-<wire x1="406.4" y1="101.6" x2="396.4268" y2="81.365" width="0" layer="19" extent="16-16"/>
 </signal>
 <signal name="A11">
@@
 <contactref element="U7" pad="14"/>
 <contactref element="X9" pad="A5"/>
-<wire x1="396.4268" y1="80.065" x2="406.4" y2="93.98" width="0" layer="19" extent="16-16"/>
-<wire x1="335.4668" y1="80.065" x2="396.4268" y2="80.065" width="0" layer="19" extent="16-16"/>
-<wire x1="274.5068" y1="80.065" x2="335.4668" y2="80.065" width="0" layer="19" extent="16-16"/>
-<wire x1="213.5468" y1="80.065" x2="274.5068" y2="80.065" width="0" layer="19" extent="16-16"/>
-<wire x1="152.5868" y1="80.065" x2="213.5468" y2="80.065" width="0" layer="19" extent="16-16"/>
+<wire x1="399.034" y1="81.534" x2="399.034" y2="93.98" width="0.3048" layer="16"/>
+<wire x1="399.034" y1="93.98" x2="400.304" y2="95.25" width="0.3048" layer="16"/>
+<wire x1="400.304" y1="95.25" x2="405.13" y2="95.25" width="0.3048" layer="16"/>
+<wire x1="405.13" y1="95.25" x2="406.4" y2="93.98" width="0.3048" layer="16"/>
+<wire x1="396.4268" y1="80.065" x2="397.565" y2="80.065" width="0.3048" layer="16"/>
+<wire x1="397.565" y1="80.065" x2="399.034" y2="81.534" width="0.3048" layer="16"/>
 <wire x1="91.6268" y1="80.065" x2="152.5868" y2="80.065" width="0" layer="19" extent="16-16"/>
 <wire x1="30.6668" y1="80.065" x2="91.6268" y2="80.065" width="0" layer="19" extent="16-16"/>
+<wire x1="213.5468" y1="80.065" x2="152.5868" y2="80.065" width="0" layer="19" extent="16-16"/>
+<wire x1="274.5068" y1="80.065" x2="213.5468" y2="80.065" width="0" layer="19" extent="16-16"/>
+<wire x1="335.4668" y1="80.065" x2="274.5068" y2="80.065" width="0" layer="19" extent="16-16"/>
+<wire x1="396.4268" y1="80.065" x2="335.4668" y2="80.065" width="0" layer="19" extent="16-16"/>
 </signal>
 <signal name="C3">
@@
 <wire x1="323.85" y1="100.33" x2="322.58" y2="99.06" width="0.4064" layer="2"/>
 <wire x1="322.58" y1="99.06" x2="320.04" y2="99.06" width="0.4064" layer="2"/>
-<wire x1="381" y1="99.06" x2="406.4" y2="99.06" width="0" layer="19" extent="1-1"/>
+<wire x1="381" y1="99.06" x2="383.667" y2="99.06" width="0.3048" layer="2"/>
+<wire x1="383.667" y1="99.06" x2="384.937" y2="100.33" width="0.3048" layer="2"/>
+<wire x1="384.937" y1="100.33" x2="405.13" y2="100.33" width="0.3048" layer="2"/>
+<wire x1="405.13" y1="100.33" x2="406.4" y2="99.06" width="0.3048" layer="2"/>
 </signal>
 <signal name="A4">
@@
 <contactref element="U7" pad="13"/>
 <contactref element="X9" pad="C2"/>
-<wire x1="396.4268" y1="80.715" x2="401.32" y2="101.6" width="0" layer="19" extent="16-16"/>
+<wire x1="398.399" y1="81.788" x2="398.399" y2="98.679" width="0.3048" layer="16"/>
+<wire x1="396.4268" y1="80.715" x2="397.326" y2="80.715" width="0.3048" layer="16"/>
+<wire x1="397.326" y1="80.715" x2="398.399" y2="81.788" width="0.3048" layer="16"/>
 <wire x1="335.4668" y1="80.715" x2="396.4268" y2="80.715" width="0" layer="19" extent="16-16"/>
 <wire x1="274.5068" y1="80.715" x2="335.4668" y2="80.715" width="0" layer="19" extent="16-16"/>
@@
 <wire x1="91.6268" y1="80.715" x2="152.5868" y2="80.715" width="0" layer="19" extent="16-16"/>
 <wire x1="30.6668" y1="80.715" x2="91.6268" y2="80.715" width="0" layer="19" extent="16-16"/>
+<wire x1="398.399" y1="98.679" x2="401.32" y2="101.6" width="0.3048" layer="16"/>
 </signal>
 <signal name="C11">
@@
 <contactref element="U7" pad="15"/>
 <contactref element="X9" pad="C5"/>
-<wire x1="396.4268" y1="79.415" x2="401.32" y2="93.98" width="0" layer="19" extent="16-16"/>
-<wire x1="335.4668" y1="79.415" x2="396.4268" y2="79.415" width="0" layer="19" extent="16-16"/>
-<wire x1="274.5068" y1="79.415" x2="335.4668" y2="79.415" width="0" layer="19" extent="16-16"/>
-<wire x1="213.5468" y1="79.415" x2="274.5068" y2="79.415" width="0" layer="19" extent="16-16"/>
-<wire x1="152.5868" y1="79.415" x2="213.5468" y2="79.415" width="0" layer="19" extent="16-16"/>
+<wire x1="396.4268" y1="79.415" x2="397.804" y2="79.415" width="0.3048" layer="16"/>
+<wire x1="397.804" y1="79.415" x2="399.796" y2="81.407" width="0.3048" layer="16"/>
+<wire x1="399.796" y1="81.407" x2="399.796" y2="92.456" width="0.3048" layer="16"/>
+<wire x1="399.796" y1="92.456" x2="401.32" y2="93.98" width="0.3048" layer="16"/>
 <wire x1="91.6268" y1="79.415" x2="152.5868" y2="79.415" width="0" layer="19" extent="16-16"/>
 <wire x1="30.6668" y1="79.415" x2="91.6268" y2="79.415" width="0" layer="19" extent="16-16"/>
+<wire x1="213.5468" y1="79.415" x2="152.5868" y2="79.415" width="0" layer="19" extent="16-16"/>
+<wire x1="274.5068" y1="79.415" x2="213.5468" y2="79.415" width="0" layer="19" extent="16-16"/>
+<wire x1="335.4668" y1="79.415" x2="274.5068" y2="79.415" width="0" layer="19" extent="16-16"/>
+<wire x1="396.4268" y1="79.415" x2="335.4668" y2="79.415" width="0" layer="19" extent="16-16"/>
 </signal>
 <signal name="CLK_0">
@@
 <contactref element="U7" pad="16"/>
 <contactref element="X9" pad="C10"/>
-<wire x1="401.32" y1="81.28" x2="400.05" y2="81.28" width="0.3048" layer="16"/>
+<wire x1="401.32" y1="81.28" x2="400.685" y2="81.28" width="0.3048" layer="16"/>
 <wire x1="396.4268" y1="78.765" x2="396.4518" y2="78.74" width="0.3048" layer="16"/>
 <wire x1="396.4518" y1="78.74" x2="398.145" y2="78.74" width="0.3048" layer="16"/>
-<wire x1="398.145" y1="78.74" x2="398.78" y2="79.375" width="0.3048" layer="16"/>
-<wire x1="398.78" y1="79.375" x2="398.78" y2="80.01" width="0.3048" layer="16"/>
-<wire x1="398.78" y1="80.01" x2="400.05" y2="81.28" width="0.3048" layer="16"/>
+<wire x1="398.145" y1="78.74" x2="400.685" y2="81.28" width="0.3048" layer="16"/>
 </signal>
 <signal name="CS_6">
@@
 <wire x1="405.13" y1="81.28" x2="403.86" y2="80.01" width="0.3048" layer="16"/>
 <wire x1="403.86" y1="80.01" x2="400.685" y2="80.01" width="0.3048" layer="16"/>
-<wire x1="400.685" y1="80.01" x2="400.05" y2="80.01" width="0" layer="19" extent="1-16"/>
 <wire x1="398.77" y1="78.115" x2="396.4268" y2="78.115" width="0.3048" layer="16"/>
 <wire x1="398.77" y1="78.115" x2="398.78" y2="78.105" width="0.3048" layer="16"/>

Commit message: Confused about L2 inductor and 5V supply for the TBX0108
Routing:
- net C11: track 17.4 -> 491.4 mm, vias 0 -> 12
- net A11: track 24.1 -> 476.9 mm, vias 0 -> 11
- net C10: track 23.4 -> 468.8 mm, vias 0 -> 11
- net A10: track 30.3 -> 434.0 mm, vias 0 -> 8
- net MISO_4: track 0.00 -> 159.5 mm, vias 0 -> 2
- net CLK_4: track 0.00 -> 156.6 mm, vias 0 -> 2
- net MOSI_4: track 0.00 -> 156.3 mm, vias 0 -> 2
- net CS_4: track 0.00 -> 149.0 mm, vias 0 -> 2
- net C32: track 246.8 -> 372.1 mm
- net A32: track 248.0 -> 372.1 mm
- net CLK_5: track 0.00 -> 95.7 mm, vias 0 -> 2
- net MISO_5: track 0.00 -> 92.8 mm, vias 0 -> 2
- net CS_5: track 0.00 -> 88.4 mm, vias 0 -> 2
- net MOSI_5: track 0.00 -> 86.9 mm, vias 0 -> 2
- net A7: track 372.1 -> 398.5 mm
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- added copper zone on layer 14, net +15V
- added copper zone on layer 15, net -15V
- added copper zone on layer 1, net GND
- added copper zone on layer 14, net GND
- added copper zone on layer 15, net GND
- added copper zone on layer 3, net GND
